Commit message: 对urdf文件进行了修改，添加了手臂模型

File: freehand_description/urdf/freehand_description_backup.urdf (robot description, URDF)
Before this commit: robot freehand_with_ur10, 46 links, 45 joints
Links:
- removed link robot_base_link
- removed link robot_ee_link
- removed link robot_forearm_link
- removed link robot_shoulder_link
- removed link robot_upper_arm_link
- removed link robot_wrist_1_link
- removed link robot_wrist_2_link
- removed link robot_wrist_3_link
- removed link world
Joints:
- removed joint arm_gripper_joint
- removed joint robot_ee_fixed_joint
- removed joint robot_elbow_joint
- removed joint robot_shoulder_lift_joint
- removed joint robot_shoulder_pan_joint
- removed joint robot_wrist_1_joint
- removed joint robot_wrist_2_joint
- removed joint robot_wrist_3_joint
- removed joint world_arm_joint
