Commit message: 添加了tacto进行触觉可视化,然后揽线的仿真测试完成了

File: otherModel/urdf/coffee_cup.urdf (robot description, URDF)
Before this commit: robot apple, 1 links, 0 joints
Links:
- link baseLink: geometry collision mesh filename=../meshes/notextures/coffee_cup.obj scale=0.001 0.001 0.001; visual mesh filename=../meshes/notextures/coffee_cup.obj scale=0.001 0.001 0.001
